Commit message: Rename robile configurations and brick names

File: robots/4_wheel_config.urdf.xacro (robot description, xacro)
@@ -3,26 +3,25 @@
     <!-- Include desired robile modules -->
     <xacro:include filename="$(find robile_description)/urdf/robile_modules/robile_active_wheel.urdf.xacro" />
-    <xacro:include filename="$(find robile_description)/urdf/robile_modules/robile_passive_wheel.urdf.xacro" />
     <xacro:include filename="$(find robile_description)/urdf/robile_modules/robile_cpu.urdf.xacro" />
     <xacro:include filename="$(find robile_description)/urdf/robile_modules/robile_master_battery.urdf.xacro" />
     <link name="base_link"/>
     <!-- Build platform using robile modules -->
-    <xacro:robile_passive_wheel name="front_right_robile" parent="base_link">
+    <xacro:robile_active_wheel name="robile_1" parent="base_link">
         <origin xyz="0.233 -0.1165 0.05" rpy="0.0 0.0 0.0"/>
-    </xacro:robile_passive_wheel>
-    <xacro:robile_active_wheel name="rear_right_robile" parent="base_link">
+    </xacro:robile_active_wheel>
+    <xacro:robile_active_wheel name="robile_2" parent="base_link">
+        <origin xyz="0.233 0.1165 0.05" rpy="0.0 0.0 0.0"/>
+    </xacro:robile_active_wheel>
+    <xacro:robile_cpu name="robile_3" parent="base_link">
+        <origin xyz="0.0 -0.1165 0.05" rpy="0.0 0.0 0.0"/>
+    </xacro:robile_cpu>
+    <xacro:robile_master_battery name="robile_4" parent="base_link">
+        <origin xyz="0.0 0.1165 0.05" rpy="0.0 0.0 0.0"/>
+    </xacro:robile_master_battery>
+    <xacro:robile_active_wheel name="robile_5" parent="base_link">
         <origin xyz="-0.233 -0.1165 0.05" rpy="0.0 0.0 0.0"/>
     </xacro:robile_active_wheel>
-    <xacro:robile_master_battery name="battery_robile" parent="base_link">
-        <origin xyz="0.0 0.1165 0.05" rpy="0.0 0.0 0.0"/>
-    </xacro:robile_master_battery>
-    <xacro:robile_cpu name="cpu_robile" parent="base_link">
-        <origin xyz="0.0 -0.1165 0.05" rpy="0.0 0.0 0.0"/>
-    </xacro:robile_cpu>
-    <xacro:robile_active_wheel name="rear_left_robile" parent="base_link">
+    <xacro:robile_active_wheel name="robile_6" parent="base_link">
         <origin xyz="-0.233 0.1165 0.05" rpy="0.0 0.0 0.0"/>
     </xacro:robile_active_wheel>
-    <xacro:robile_passive_wheel name="front_left_robile" parent="base_link">
-        <origin xyz="0.233 0.1165 0.05" rpy="0.0 0.0 0.0"/>
-    </xacro:robile_passive_wheel>
 </robot>
