Commit message: Fix robile positions in 2 and 4 wheel configs

File: robots/2_wheel_config.urdf.xacro (robot description, xacro)
@@ -9,20 +9,20 @@
     <!-- Build platform using robile modules -->
     <xacro:robile_passive_wheel name="robile_1" parent="base_link">
+        <origin xyz="0.233 0.1165 0.05" rpy="0.0 0.0 0.0"/>
+    </xacro:robile_passive_wheel>
+    <xacro:robile_passive_wheel name="robile_2" parent="base_link">
         <origin xyz="0.233 -0.1165 0.05" rpy="0.0 0.0 0.0"/>
     </xacro:robile_passive_wheel>
-    <xacro:robile_passive_wheel name="robile_2" parent="base_link">
-        <origin xyz="0.233 0.1165 0.05" rpy="0.0 0.0 0.0"/>
-    </xacro:robile_passive_wheel>
     <xacro:robile_cpu name="robile_3" parent="base_link">
-        <origin xyz="0.0 -0.1165 0.05" rpy="0.0 0.0 0.0"/>
+        <origin xyz="0.0 0.1165 0.05" rpy="0.0 0.0 0.0"/>
     </xacro:robile_cpu>
     <xacro:robile_master_battery name="robile_4" parent="base_link">
-        <origin xyz="0.0 0.1165 0.05" rpy="0.0 0.0 0.0"/>
+        <origin xyz="0.0 -0.1165 0.05" rpy="0.0 0.0 0.0"/>
     </xacro:robile_master_battery>
     <xacro:robile_active_wheel name="robile_5" parent="base_link">
+        <origin xyz="-0.233 0.1165 0.05" rpy="0.0 0.0 0.0"/>
+    </xacro:robile_active_wheel>
+    <xacro:robile_active_wheel name="robile_6" parent="base_link">
         <origin xyz="-0.233 -0.1165 0.05" rpy="0.0 0.0 0.0"/>
     </xacro:robile_active_wheel>
-    <xacro:robile_active_wheel name="robile_6" parent="base_link">
-        <origin xyz="-0.233 0.1165 0.05" rpy="0.0 0.0 0.0"/>
-    </xacro:robile_active_wheel>
 </robot>

File: robots/4_wheel_config.urdf.xacro (robot description, xacro)
@@ -8,20 +8,20 @@
     <!-- Build platform using robile modules -->
     <xacro:robile_active_wheel name="robile_1" parent="base_link">
+        <origin xyz="0.233 0.1165 0.05" rpy="0.0 0.0 0.0"/>
+    </xacro:robile_active_wheel>
+    <xacro:robile_active_wheel name="robile_2" parent="base_link">
         <origin xyz="0.233 -0.1165 0.05" rpy="0.0 0.0 0.0"/>
     </xacro:robile_active_wheel>
-    <xacro:robile_active_wheel name="robile_2" parent="base_link">
-        <origin xyz="0.233 0.1165 0.05" rpy="0.0 0.0 0.0"/>
-    </xacro:robile_active_wheel>
     <xacro:robile_cpu name="robile_3" parent="base_link">
-        <origin xyz="0.0 -0.1165 0.05" rpy="0.0 0.0 0.0"/>
+        <origin xyz="0.0 0.1165 0.05" rpy="0.0 0.0 0.0"/>
     </xacro:robile_cpu>
     <xacro:robile_master_battery name="robile_4" parent="base_link">
-        <origin xyz="0.0 0.1165 0.05" rpy="0.0 0.0 0.0"/>
+        <origin xyz="0.0 -0.1165 0.05" rpy="0.0 0.0 0.0"/>
     </xacro:robile_master_battery>
     <xacro:robile_active_wheel name="robile_5" parent="base_link">
+        <origin xyz="-0.233 0.1165 0.05" rpy="0.0 0.0 0.0"/>
+    </xacro:robile_active_wheel>
+    <xacro:robile_active_wheel name="robile_6" parent="base_link">
         <origin xyz="-0.233 -0.1165 0.05" rpy="0.0 0.0 0.0"/>
     </xacro:robile_active_wheel>
-    <xacro:robile_active_wheel name="robile_6" parent="base_link">
-        <origin xyz="-0.233 0.1165 0.05" rpy="0.0 0.0 0.0"/>
-    </xacro:robile_active_wheel>
 </robot>

Commit message: Rename robile_module -> robile_brick

File: robots/2_wheel_config.urdf.xacro (robot description, xacro)
@@ -30,28 +30,28 @@
 -->
 <robot xmlns:xacro="http://ros.org/wiki/xacro" name="2_wheel_config" >
-    <!-- Include desired robile modules -->
-    <xacro:include filename="$(find robile_description)/urdf/robile_modules/robile_active_wheel.urdf.xacro" />
-    <xacro:include filename="$(find robile_description)/urdf/robile_modules/robile_passive_wheel.urdf.xacro" />
-    <xacro:include filename="$(find robile_description)/urdf/robile_modules/robile_cpu.urdf.xacro" />
-    <xacro:include filename="$(find robile_description)/urdf/robile_modules/robile_master_battery.urdf.xacro" />
+    <!-- Include desired robile bricks -->
+    <xacro:include filename="$(find robile_description)/urdf/robile_bricks/robile_active_wheel_brick.urdf.xacro" />
+    <xacro:include filename="$(find robile_description)/urdf/robile_bricks/robile_passive_wheel_brick.urdf.xacro" />
+    <xacro:include filename="$(find robile_description)/urdf/robile_bricks/robile_cpu_brick.urdf.xacro" />
+    <xacro:include filename="$(find robile_description)/urdf/robile_bricks/robile_master_battery_brick.urdf.xacro" />
     <link name="base_link"/>
-    <!-- Build platform using robile modules -->
-    <xacro:robile_passive_wheel name="robile_1" parent="base_link">
+    <!-- Build platform using robile bricks -->
+    <xacro:robile_passive_wheel_brick name="robile_1" parent="base_link">
         <origin xyz="0.233 0.1165 0.05" rpy="0.0 0.0 0.0"/>
-    </xacro:robile_passive_wheel>
-    <xacro:robile_passive_wheel name="robile_2" parent="base_link">
+    </xacro:robile_passive_wheel_brick>
+    <xacro:robile_passive_wheel_brick name="robile_2" parent="base_link">
         <origin xyz="0.233 -0.1165 0.05" rpy="0.0 0.0 0.0"/>
-    </xacro:robile_passive_wheel>
-    <xacro:robile_cpu name="robile_3" parent="base_link">
+    </xacro:robile_passive_wheel_brick>
+    <xacro:robile_cpu_brick name="robile_3" parent="base_link">
         <origin xyz="0.0 0.1165 0.05" rpy="0.0 0.0 0.0"/>
-    </xacro:robile_cpu>
-    <xacro:robile_master_battery name="robile_4" parent="base_link">
+    </xacro:robile_cpu_brick>
+    <xacro:robile_master_battery_brick name="robile_4" parent="base_link">
         <origin xyz="0.0 -0.1165 0.05" rpy="0.0 0.0 0.0"/>
-    </xacro:robile_master_battery>
-    <xacro:robile_active_wheel name="robile_5" parent="base_link">
+    </xacro:robile_master_battery_brick>
+    <xacro:robile_active_wheel_brick name="robile_5" parent="base_link">
         <origin xyz="-0.233 0.1165 0.05" rpy="0.0 0.0 0.0"/>
-    </xacro:robile_active_wheel>
-    <xacro:robile_active_wheel name="robile_6" parent="base_link">
+    </xacro:robile_active_wheel_brick>
+    <xacro:robile_active_wheel_brick name="robile_6" parent="base_link">
         <origin xyz="-0.233 -0.1165 0.05" rpy="0.0 0.0 0.0"/>
-    </xacro:robile_active_wheel>
+    </xacro:robile_active_wheel_brick>
 </robot>

File: robots/4_wheel_config.urdf.xacro (robot description, xacro)
@@ -30,27 +30,27 @@
 -->
 <robot xmlns:xacro="http://ros.org/wiki/xacro" name="4_wheel_config" >
-    <!-- Include desired robile modules -->
-    <xacro:include filename="$(find robile_description)/urdf/robile_modules/robile_active_wheel.urdf.xacro" />
-    <xacro:include filename="$(find robile_description)/urdf/robile_modules/robile_cpu.urdf.xacro" />
-    <xacro:include filename="$(find robile_description)/urdf/robile_modules/robile_master_battery.urdf.xacro" />
+    <!-- Include desired robile bricks -->
+    <xacro:include filename="$(find robile_description)/urdf/robile_bricks/robile_active_wheel_brick.urdf.xacro" />
+    <xacro:include filename="$(find robile_description)/urdf/robile_bricks/robile_cpu_brick.urdf.xacro" />
+    <xacro:include filename="$(find robile_description)/urdf/robile_bricks/robile_master_battery_brick.urdf.xacro" />
     <link name="base_link"/>
-    <!-- Build platform using robile modules -->
-    <xacro:robile_active_wheel name="robile_1" parent="base_link">
+    <!-- Build platform using robile bricks -->
+    <xacro:robile_active_wheel_brick name="robile_1" parent="base_link">
         <origin xyz="0.233 0.1165 0.05" rpy="0.0 0.0 0.0"/>
-    </xacro:robile_active_wheel>
-    <xacro:robile_active_wheel name="robile_2" parent="base_link">
+    </xacro:robile_active_wheel_brick>
+    <xacro:robile_active_wheel_brick name="robile_2" parent="base_link">
         <origin xyz="0.233 -0.1165 0.05" rpy="0.0 0.0 0.0"/>
-    </xacro:robile_active_wheel>
-    <xacro:robile_cpu name="robile_3" parent="base_link">
+    </xacro:robile_active_wheel_brick>
+    <xacro:robile_cpu_brick name="robile_3" parent="base_link">
         <origin xyz="0.0 0.1165 0.05" rpy="0.0 0.0 0.0"/>
-    </xacro:robile_cpu>
-    <xacro:robile_master_battery name="robile_4" parent="base_link">
+    </xacro:robile_cpu_brick>
+    <xacro:robile_master_battery_brick name="robile_4" parent="base_link">
         <origin xyz="0.0 -0.1165 0.05" rpy="0.0 0.0 0.0"/>
-    </xacro:robile_master_battery>
-    <xacro:robile_active_wheel name="robile_5" parent="base_link">
+    </xacro:robile_master_battery_brick>
+    <xacro:robile_active_wheel_brick name="robile_5" parent="base_link">
         <origin xyz="-0.233 0.1165 0.05" rpy="0.0 0.0 0.0"/>
-    </xacro:robile_active_wheel>
-    <xacro:robile_active_wheel name="robile_6" parent="base_link">
+    </xacro:robile_active_wheel_brick>
+    <xacro:robile_active_wheel_brick name="robile_6" parent="base_link">
         <origin xyz="-0.233 -0.1165 0.05" rpy="0.0 0.0 0.0"/>
-    </xacro:robile_active_wheel>
+    </xacro:robile_active_wheel_brick>
 </robot>

File: robots/6_wheel_config.urdf.xacro (robot description, xacro)
@@ -30,55 +30,55 @@
 -->
 <robot xmlns:xacro="http://ros.org/wiki/xacro" name="6_wheel_config" >
-    <!-- Include desired robile modules -->
-    <xacro:include filename="$(find robile_description)/urdf/robile_modules/robile_active_wheel.urdf.xacro" />
-    <xacro:include filename="$(find robile_description)/urdf/robile_modules/robile_cpu.urdf.xacro" />
-    <xacro:include filename="$(find robile_description)/urdf/robile_modules/robile_master_battery.urdf.xacro" />
-    <xacro:include filename="$(find robile_description)/urdf/robile_modules/robile_empty.urdf.xacro" />
+    <!-- Include desired robile bricks -->
+    <xacro:include filename="$(find robile_description)/urdf/robile_bricks/robile_active_wheel_brick.urdf.xacro" />
+    <xacro:include filename="$(find robile_description)/urdf/robile_bricks/robile_cpu_brick.urdf.xacro" />
+    <xacro:include filename="$(find robile_description)/urdf/robile_bricks/robile_master_battery_brick.urdf.xacro" />
+    <xacro:include filename="$(find robile_description)/urdf/robile_bricks/robile_empty_brick.urdf.xacro" />
     <link name="base_link"/>
-    <!-- Build platform using robile modules -->
-    <xacro:robile_active_wheel name="robile_1" parent="base_link">
+    <!-- Build platform using robile bricks -->
+    <xacro:robile_active_wheel_brick name="robile_1" parent="base_link">
         <origin xyz="0.233 0.466 0.05" rpy="0.0 0.0 0.0"/>
-    </xacro:robile_active_wheel>
-    <xacro:robile_empty name="robile_2" parent="base_link">
+    </xacro:robile_active_wheel_brick>
+    <xacro:robile_empty_brick name="robile_2" parent="base_link">
         <origin xyz="0 0.466 0.05" rpy="0.0 0.0 0.0"/>
-    </xacro:robile_empty>
-    <xacro:robile_active_wheel name="robile_3" parent="base_link">
+    </xacro:robile_empty_brick>
+    <xacro:robile_active_wheel_brick name="robile_3" parent="base_link">
         <origin xyz="-0.233 0.466 0.05" rpy="0.0 0.0 0.0"/>
-    </xacro:robile_active_wheel>
-    <xacro:robile_empty name="robile_4" parent="base_link">
+    </xacro:robile_active_wheel_brick>
+    <xacro:robile_empty_brick name="robile_4" parent="base_link">
         <origin xyz="0.233 0.233 0.05" rpy="0.0 0.0 0.0"/>
-    </xacro:robile_empty>
-    <xacro:robile_master_battery name="robile_5" parent="base_link">
+    </xacro:robile_empty_brick>
+    <xacro:robile_master_battery_brick name="robile_5" parent="base_link">
         <origin xyz="0 0.233 0.05" rpy="0.0 0.0 0.0"/>
-    </xacro:robile_master_battery>
-    <xacro:robile_empty name="robile_6" parent="base_link">
+    </xacro:robile_master_battery_brick>
+    <xacro:robile_empty_brick name="robile_6" parent="base_link">
         <origin xyz="-0.233 0.233 0.05" rpy="0.0 0.0 0.0"/>
-    </xacro:robile_empty>
-    <xacro:robile_active_wheel name="robile_7" parent="base_link">
+    </xacro:robile_empty_brick>
+    <xacro:robile_active_wheel_brick name="robile_7" parent="base_link">
         <origin xyz="0.233 0 0.05" rpy="0.0 0.0 0.0"/>
-    </xacro:robile_active_wheel>
-    <xacro:robile_empty name="robile_8" parent="base_link">
+    </xacro:robile_active_wheel_brick>
+    <xacro:robile_empty_brick name="robile_8" parent="base_link">
         <origin xyz="0 0 0.05" rpy="0.0 0.0 0.0"/>
-    </xacro:robile_empty>
-    <xacro:robile_active_wheel name="robile_9" parent="base_link">
+    </xacro:robile_empty_brick>
+    <xacro:robile_active_wheel_brick name="robile_9" parent="base_link">
         <origin xyz="-0.233 0 0.05" rpy="0.0 0.0 0.0"/>
-    </xacro:robile_active_wheel>
-    <xacro:robile_empty name="robile_10" parent="base_link">
+    </xacro:robile_active_wheel_brick>
+    <xacro:robile_empty_brick name="robile_10" parent="base_link">
         <origin xyz="0.233 -0.233 0.05" rpy="0.0 0.0 0.0"/>
-    </xacro:robile_empty>
-    <xacro:robile_cpu name="robile_11" parent="base_link">
+    </xacro:robile_empty_brick>
+    <xacro:robile_cpu_brick name="robile_11" parent="base_link">
         <origin xyz="0 -0.233 0.05" rpy="0.0 0.0 0.0"/>
-    </xacro:robile_cpu>
-    <xacro:robile_empty name="robile_12" parent="base_link">
+    </xacro:robile_cpu_brick>
+    <xacro:robile_empty_brick name="robile_12" parent="base_link">
         <origin xyz="-0.233 -0.233 0.05" rpy="0.0 0.0 0.0"/>
-    </xacro:robile_empty>
-    <xacro:robile_active_wheel name="robile_13" parent="base_link">
+    </xacro:robile_empty_brick>
+    <xacro:robile_active_wheel_brick name="robile_13" parent="base_link">
         <origin xyz="0.233 -0.466 0.05" rpy="0.0 0.0 0.0"/>
-    </xacro:robile_active_wheel>
-    <xacro:robile_empty name="robile_14" parent="base_link">
+    </xacro:robile_active_wheel_brick>
+    <xacro:robile_empty_brick name="robile_14" parent="base_link">
         <origin xyz="0 -0.466 0.05" rpy="0.0 0.0 0.0"/>
-    </xacro:robile_empty>
-    <xacro:robile_active_wheel name="robile_15" parent="base_link">
+    </xacro:robile_empty_brick>
+    <xacro:robile_active_wheel_brick name="robile_15" parent="base_link">
         <origin xyz="-0.233 -0.466 0.05" rpy="0.0 0.0 0.0"/>
-    </xacro:robile_active_wheel>
+    </xacro:robile_active_wheel_brick>
 </robot>

File: urdf/base_macros/robile_body.urdf.xacro (robot description, xacro)
@@ -33,5 +33,5 @@
         <!-- Include required xacro files -->
         <xacro:include filename="$(find robile_description)/urdf/base_macros/common.xacro" />
-        <!-- Properties for a robile module -->
+        <!-- Properties for a robile brick -->
         <xacro:property name="robile_size_x" value="0.233"/>
         <xacro:property name="robile_size_y" value="0.233"/>

File: urdf/robile_bricks/robile_active_wheel_brick.urdf.xacro (robot description, xacro)
@@ -30,8 +30,8 @@
 -->
 <robot xmlns:xacro="http://www.ros.org/wiki/xacro">
-    <xacro:macro name="robile_passive_wheel" params="name parent *origin">
+    <xacro:macro name="robile_active_wheel_brick" params="name parent *origin">
         <!-- Include xacro files-->
         <xacro:include filename="$(find robile_description)/urdf/base_macros/robile_body.urdf.xacro" />
-        <xacro:include filename="$(find robile_description)/urdf/base_macros/caster_wheel.urdf.xacro" />
+        <xacro:include filename="$(find robile_description)/urdf/base_macros/kelo_drive.urdf.xacro" />
         <joint name="${name}_joint" type="fixed">
             <xacro:insert_block name="origin" />
@@ -39,8 +39,8 @@
             <child link="${name}_link" />
         </joint>
-        <xacro:robile_body name="${name}" with_wheel="true" color="blue"/>
-        <xacro:caster_wheel name="${name}_caster_wheel" parent="${name}_link">
+        <xacro:robile_body name="${name}" with_wheel="true" color="red"/>
+        <xacro:kelo_drive name="${name}_drive" parent="${name}_link">
             <origin xyz="0 0 0" rpy="0 0 0.0"/>
-        </xacro:caster_wheel>
+        </xacro:kelo_drive>
     </xacro:macro>
 </robot>

File: urdf/robile_bricks/robile_cpu_brick.urdf.xacro (robot description, xacro)
@@ -30,5 +30,5 @@
 -->
 <robot xmlns:xacro="http://www.ros.org/wiki/xacro">
-    <xacro:macro name="robile_master_battery" params="name parent *origin">
+    <xacro:macro name="robile_cpu_brick" params="name parent *origin">
         <xacro:include filename="$(find robile_description)/urdf/base_macros/robile_body.urdf.xacro" />
         <joint name="${name}_joint" type="fixed">
@@ -37,5 +37,5 @@
             <child link="${name}_link" />
         </joint>
-        <xacro:robile_body name="${name}" color="green"/>
+        <xacro:robile_body name="${name}"/>
     </xacro:macro>
 </robot>

File: urdf/robile_bricks/robile_empty_brick.urdf.xacro (robot description, xacro)
@@ -30,5 +30,5 @@
 -->
 <robot xmlns:xacro="http://www.ros.org/wiki/xacro">
-    <xacro:macro name="robile_empty" params="name parent *origin">
+    <xacro:macro name="robile_empty_brick" params="name parent *origin">
         <xacro:include filename="$(find robile_description)/urdf/base_macros/robile_body.urdf.xacro" />
         <joint name="${name}_joint" type="fixed">

File: urdf/robile_bricks/robile_master_battery_brick.urdf.xacro (robot description, xacro)
@@ -30,8 +30,6 @@
 -->
 <robot xmlns:xacro="http://www.ros.org/wiki/xacro">
-    <xacro:macro name="robile_active_wheel" params="name parent *origin">
-        <!-- Include xacro files-->
+    <xacro:macro name="robile_master_battery_brick" params="name parent *origin">
         <xacro:include filename="$(find robile_description)/urdf/base_macros/robile_body.urdf.xacro" />
-        <xacro:include filename="$(find robile_description)/urdf/base_macros/kelo_drive.urdf.xacro" />
         <joint name="${name}_joint" type="fixed">
             <xacro:insert_block name="origin" />
@@ -39,8 +37,5 @@
             <child link="${name}_link" />
         </joint>
-        <xacro:robile_body name="${name}" with_wheel="true" color="red"/>
-        <xacro:kelo_drive name="${name}_drive" parent="${name}_link">
-            <origin xyz="0 0 0" rpy="0 0 0.0"/>
-        </xacro:kelo_drive>
+        <xacro:robile_body name="${name}" color="green"/>
     </xacro:macro>
 </robot>

File: urdf/robile_bricks/robile_passive_wheel_brick.urdf.xacro (robot description, xacro)
@@ -30,6 +30,8 @@
 -->
 <robot xmlns:xacro="http://www.ros.org/wiki/xacro">
-    <xacro:macro name="robile_cpu" params="name parent *origin">
+    <xacro:macro name="robile_passive_wheel_brick" params="name parent *origin">
+        <!-- Include xacro files-->
         <xacro:include filename="$(find robile_description)/urdf/base_macros/robile_body.urdf.xacro" />
+        <xacro:include filename="$(find robile_description)/urdf/base_macros/caster_wheel.urdf.xacro" />
         <joint name="${name}_joint" type="fixed">
             <xacro:insert_block name="origin" />
@@ -37,5 +39,8 @@
             <child link="${name}_link" />
         </joint>
-        <xacro:robile_body name="${name}"/>
+        <xacro:robile_body name="${name}" with_wheel="true" color="blue"/>
+        <xacro:caster_wheel name="${name}_caster_wheel" parent="${name}_link">
+            <origin xyz="0 0 0" rpy="0 0 0.0"/>
+        </xacro:caster_wheel>
     </xacro:macro>
 </robot>

File: urdf/robile_bricks/robile_slave_battery_brick.urdf.xacro (robot description, xacro)
@@ -30,5 +30,5 @@
 -->
 <robot xmlns:xacro="http://www.ros.org/wiki/xacro">
-    <xacro:macro name="robile_slave_battery" params="name parent *origin">
+    <xacro:macro name="robile_slave_battery_brick" params="name parent *origin">
         <xacro:include filename="$(find robile_description)/urdf/base_macros/robile_body.urdf.xacro" />
         <joint name="${name}_joint" type="fixed">
