Commit message: Add support for disabling movable wheel joints

File: robots/2_wheel_config.urdf.xacro (robot description, xacro)
@@ -30,4 +30,5 @@
 -->
 <robot xmlns:xacro="http://ros.org/wiki/xacro" name="2_wheel_config" >
+    <xacro:arg name="movable_joints" default="true"/>
     <!-- Include desired robile bricks -->
     <xacro:include filename="$(find robile_description)/urdf/robile_bricks/robile_active_wheel_brick.urdf.xacro" />
@@ -37,8 +38,8 @@
     <link name="base_link"/>
     <!-- Build platform using robile bricks -->
-    <xacro:robile_passive_wheel_brick name="robile_1" parent="base_link">
+    <xacro:robile_passive_wheel_brick name="robile_1" parent="base_link" movable_joints="$(arg movable_joints)">
         <origin xyz="0.233 0.1165 0.05" rpy="0.0 0.0 0.0"/>
     </xacro:robile_passive_wheel_brick>
-    <xacro:robile_passive_wheel_brick name="robile_2" parent="base_link">
+    <xacro:robile_passive_wheel_brick name="robile_2" parent="base_link" movable_joints="$(arg movable_joints)">
         <origin xyz="0.233 -0.1165 0.05" rpy="0.0 0.0 0.0"/>
     </xacro:robile_passive_wheel_brick>
@@ -49,8 +50,8 @@
         <origin xyz="0.0 -0.1165 0.05" rpy="0.0 0.0 0.0"/>
     </xacro:robile_master_battery_brick>
-    <xacro:robile_active_wheel_brick name="robile_5" parent="base_link">
+    <xacro:robile_active_wheel_brick name="robile_5" parent="base_link" movable_joints="$(arg movable_joints)">
         <origin xyz="-0.233 0.1165 0.05" rpy="0.0 0.0 0.0"/>
     </xacro:robile_active_wheel_brick>
-    <xacro:robile_active_wheel_brick name="robile_6" parent="base_link">
+    <xacro:robile_active_wheel_brick name="robile_6" parent="base_link" movable_joints="$(arg movable_joints)">
         <origin xyz="-0.233 -0.1165 0.05" rpy="0.0 0.0 0.0"/>
     </xacro:robile_active_wheel_brick>

File: robots/4_wheel_config.urdf.xacro (robot description, xacro)
@@ -30,4 +30,5 @@
 -->
 <robot xmlns:xacro="http://ros.org/wiki/xacro" name="4_wheel_config" >
+    <xacro:arg name="movable_joints" default="true"/>
     <!-- Include desired robile bricks -->
     <xacro:include filename="$(find robile_description)/urdf/robile_bricks/robile_active_wheel_brick.urdf.xacro" />
@@ -36,8 +37,8 @@
     <link name="base_link"/>
     <!-- Build platform using robile bricks -->
-    <xacro:robile_active_wheel_brick name="robile_1" parent="base_link">
+    <xacro:robile_active_wheel_brick name="robile_1" parent="base_link" movable_joints="$(arg movable_joints)">
         <origin xyz="0.233 0.1165 0.05" rpy="0.0 0.0 0.0"/>
     </xacro:robile_active_wheel_brick>
-    <xacro:robile_active_wheel_brick name="robile_2" parent="base_link">
+    <xacro:robile_active_wheel_brick name="robile_2" parent="base_link" movable_joints="$(arg movable_joints)">
         <origin xyz="0.233 -0.1165 0.05" rpy="0.0 0.0 0.0"/>
     </xacro:robile_active_wheel_brick>
@@ -48,8 +49,8 @@
         <origin xyz="0.0 -0.1165 0.05" rpy="0.0 0.0 0.0"/>
     </xacro:robile_master_battery_brick>
-    <xacro:robile_active_wheel_brick name="robile_5" parent="base_link">
+    <xacro:robile_active_wheel_brick name="robile_5" parent="base_link" movable_joints="$(arg movable_joints)">
         <origin xyz="-0.233 0.1165 0.05" rpy="0.0 0.0 0.0"/>
     </xacro:robile_active_wheel_brick>
-    <xacro:robile_active_wheel_brick name="robile_6" parent="base_link">
+    <xacro:robile_active_wheel_brick name="robile_6" parent="base_link" movable_joints="$(arg movable_joints)">
         <origin xyz="-0.233 -0.1165 0.05" rpy="0.0 0.0 0.0"/>
     </xacro:robile_active_wheel_brick>

File: robots/6_wheel_config.urdf.xacro (robot description, xacro)
@@ -30,4 +30,5 @@
 -->
 <robot xmlns:xacro="http://ros.org/wiki/xacro" name="6_wheel_config" >
+    <xacro:arg name="movable_joints" default="true"/>
     <!-- Include desired robile bricks -->
     <xacro:include filename="$(find robile_description)/urdf/robile_bricks/robile_active_wheel_brick.urdf.xacro" />
@@ -37,5 +38,5 @@
     <link name="base_link"/>
     <!-- Build platform using robile bricks -->
-    <xacro:robile_active_wheel_brick name="robile_1" parent="base_link">
+    <xacro:robile_active_wheel_brick name="robile_1" parent="base_link" movable_joints="$(arg movable_joints)">
         <origin xyz="0.233 0.466 0.05" rpy="0.0 0.0 0.0"/>
     </xacro:robile_active_wheel_brick>
@@ -43,5 +44,5 @@
         <origin xyz="0 0.466 0.05" rpy="0.0 0.0 0.0"/>
     </xacro:robile_empty_brick>
-    <xacro:robile_active_wheel_brick name="robile_3" parent="base_link">
+    <xacro:robile_active_wheel_brick name="robile_3" parent="base_link" movable_joints="$(arg movable_joints)">
         <origin xyz="-0.233 0.466 0.05" rpy="0.0 0.0 0.0"/>
     </xacro:robile_active_wheel_brick>
@@ -55,5 +56,5 @@
         <origin xyz="-0.233 0.233 0.05" rpy="0.0 0.0 0.0"/>
     </xacro:robile_empty_brick>
-    <xacro:robile_active_wheel_brick name="robile_7" parent="base_link">
+    <xacro:robile_active_wheel_brick name="robile_7" parent="base_link" movable_joints="$(arg movable_joints)">
         <origin xyz="0.233 0 0.05" rpy="0.0 0.0 0.0"/>
     </xacro:robile_active_wheel_brick>
@@ -61,5 +62,5 @@
         <origin xyz="0 0 0.05" rpy="0.0 0.0 0.0"/>
     </xacro:robile_empty_brick>
-    <xacro:robile_active_wheel_brick name="robile_9" parent="base_link">
+    <xacro:robile_active_wheel_brick name="robile_9" parent="base_link" movable_joints="$(arg movable_joints)">
         <origin xyz="-0.233 0 0.05" rpy="0.0 0.0 0.0"/>
     </xacro:robile_active_wheel_brick>
@@ -73,5 +74,5 @@
         <origin xyz="-0.233 -0.233 0.05" rpy="0.0 0.0 0.0"/>
     </xacro:robile_empty_brick>
-    <xacro:robile_active_wheel_brick name="robile_13" parent="base_link">
+    <xacro:robile_active_wheel_brick name="robile_13" parent="base_link" movable_joints="$(arg movable_joints)">
         <origin xyz="0.233 -0.466 0.05" rpy="0.0 0.0 0.0"/>
     </xacro:robile_active_wheel_brick>
@@ -79,5 +80,5 @@
         <origin xyz="0 -0.466 0.05" rpy="0.0 0.0 0.0"/>
     </xacro:robile_empty_brick>
-    <xacro:robile_active_wheel_brick name="robile_15" parent="base_link">
+    <xacro:robile_active_wheel_brick name="robile_15" parent="base_link" movable_joints="$(arg movable_joints)">
         <origin xyz="-0.233 -0.466 0.05" rpy="0.0 0.0 0.0"/>
     </xacro:robile_active_wheel_brick>

File: urdf/base_macros/kelo_drive.urdf.xacro (robot description, xacro)
@@ -30,24 +30,34 @@
 -->
 <robot xmlns:xacro="http://www.ros.org/wiki/xacro">
-    <xacro:macro name="kelo_drive" params="name parent *origin">
+    <xacro:macro name="kelo_drive" params="name parent *origin movable_joints:=true">
         <xacro:include filename="$(find robile_description)/urdf/base_macros/common.xacro" />
         <xacro:include filename="$(find robile_description)/urdf/base_macros/kelo_drive_wheel.urdf.xacro" />
         <!-- PIVOT -->
-        <joint name="${name}_pivot_joint" type="continuous">
-            <xacro:insert_block name="origin" />
-            <axis xyz="0 0 1"/>
-            <parent link="${parent}"/>
-            <child link="${name}_pivot_link" />
-        </joint>
-        <transmission name="${name}_pivot_transmission">
-            <type>transmission_interface/SimpleTransmission</type>
-            <joint name="${name}_pivot_joint">
-                <hardwareInterface>hardware_interface/EffortJointInterface</hardwareInterface>
+        <xacro:if value="${movable_joints}">
+            <joint name="${name}_pivot_joint" type="continuous">
+                <xacro:insert_block name="origin" />
+                <axis xyz="0 0 1"/>
+                <parent link="${parent}"/>
+                <child link="${name}_pivot_link" />
             </joint>
-            <actuator name="${name}_pivot_motor">
-                <hardwareInterface>hardware_interface/EffortJointInterface</hardwareInterface>
-                <mechanicalReduction>1</mechanicalReduction>
-            </actuator>
-        </transmission>
+            <transmission name="${name}_pivot_transmission">
+                <type>transmission_interface/SimpleTransmission</type>
+                <joint name="${name}_pivot_joint">
+                    <hardwareInterface>hardware_interface/EffortJointInterface</hardwareInterface>
+                </joint>
+                <actuator name="${name}_pivot_motor">
+                    <hardwareInterface>hardware_interface/EffortJointInterface</hardwareInterface>
+                    <mechanicalReduction>1</mechanicalReduction>
+                </actuator>
+            </transmission>
+        </xacro:if>
+        <xacro:unless value="${movable_joints}">
+            <joint name="${name}_pivot_joint" type="fixed">
+                <xacro:insert_block name="origin" />
+                <axis xyz="0 0 1"/>
+                <parent link="${parent}"/>
+                <child link="${name}_pivot_link" />
+            </joint>
+        </xacro:unless>
         <link name="${name}_pivot_link">
             <visual>
@@ -68,9 +78,9 @@
         </link>
         <!-- LEFT HUB WHEEL -->
-        <xacro:kelo_drive_wheel name="${name}_left_hub_wheel" parent="${name}_pivot_link">
+        <xacro:kelo_drive_wheel name="${name}_left_hub_wheel" parent="${name}_pivot_link" movable_joints="${movable_joints}">
             <origin xyz="-0.01 0.039326 0.001514" rpy="0 0 0.0"/>
         </xacro:kelo_drive_wheel>
         <!-- RIGHT HUB WHEEL -->
-        <xacro:kelo_drive_wheel name="${name}_right_hub_wheel" parent="${name}_pivot_link">
+        <xacro:kelo_drive_wheel name="${name}_right_hub_wheel" parent="${name}_pivot_link" movable_joints="${movable_joints}">
             <origin xyz="-0.01 -0.039326 0.001514" rpy="0 0 0.0"/>
         </xacro:kelo_drive_wheel>

File: urdf/base_macros/kelo_drive_wheel.urdf.xacro (robot description, xacro)
@@ -30,22 +30,32 @@
 -->
 <robot xmlns:xacro="http://www.ros.org/wiki/xacro">
-    <xacro:macro name="kelo_drive_wheel" params="name parent *origin">
+    <xacro:macro name="kelo_drive_wheel" params="name parent *origin movable_joints:=true">
         <xacro:include filename="$(find robile_description)/urdf/base_macros/common.xacro" />
-        <joint name="${name}_joint" type="continuous">
-            <xacro:insert_block name="origin" />
-            <axis xyz="0 1 0"/>
-            <parent link="${parent}"/>
-            <child link="${name}_link" />
-        </joint>
-        <transmission name="${name}_transmission">
-            <type>transmission_interface/SimpleTransmission</type>
-            <joint name="${name}_joint">
-                <hardwareInterface>hardware_interface/EffortJointInterface</hardwareInterface>
+        <xacro:if value="${movable_joints}">
+            <joint name="${name}_joint" type="continuous">
+                <xacro:insert_block name="origin" />
+                <axis xyz="0 1 0"/>
+                <parent link="${parent}"/>
+                <child link="${name}_link" />
             </joint>
-            <actuator name="${name}_motor">
-                <hardwareInterface>hardware_interface/EffortJointInterface</hardwareInterface>
-                <mechanicalReduction>1</mechanicalReduction>
-            </actuator>
-        </transmission>
+            <transmission name="${name}_transmission">
+                <type>transmission_interface/SimpleTransmission</type>
+                <joint name="${name}_joint">
+                    <hardwareInterface>hardware_interface/EffortJointInterface</hardwareInterface>
+                </joint>
+                <actuator name="${name}_motor">
+                    <hardwareInterface>hardware_interface/EffortJointInterface</hardwareInterface>
+                    <mechanicalReduction>1</mechanicalReduction>
+                </actuator>
+            </transmission>
+        </xacro:if>
+        <xacro:unless value="${movable_joints}">
+            <joint name="${name}_joint" type="fixed">
+                <xacro:insert_block name="origin" />
+                <axis xyz="0 1 0"/>
+                <parent link="${parent}"/>
+                <child link="${name}_link" />
+            </joint>
+        </xacro:unless>
         <link name="${name}_link">
             <visual>

File: urdf/base_macros/passive_caster_wheel.urdf.xacro (robot description, xacro)
@@ -30,23 +30,33 @@
 -->
 <robot xmlns:xacro="http://www.ros.org/wiki/xacro">
-    <xacro:macro name="passive_caster_wheel" params="name parent *origin">
+    <xacro:macro name="passive_caster_wheel" params="name parent *origin movable_joints:=true">
         <xacro:include filename="$(find robile_description)/urdf/base_macros/common.xacro" />
         <!-- PIVOT -->
-        <joint name="${name}_pivot_caster_joint" type="continuous">
-            <xacro:insert_block name="origin" />
-            <axis xyz="0 0 1"/>
-            <parent link="${parent}"/>
-            <child link="${name}_pivot_link" />
-        </joint>
-        <transmission name="${name}_pivot_transmission">
-            <type>transmission_interface/SimpleTransmission</type>
-            <joint name="${name}_pivot_caster_joint">
-                <hardwareInterface>hardware_interface/EffortJointInterface</hardwareInterface>
+        <xacro:if value="${movable_joints}">
+            <joint name="${name}_pivot_caster_joint" type="continuous">
+                <xacro:insert_block name="origin" />
+                <axis xyz="0 0 1"/>
+                <parent link="${parent}"/>
+                <child link="${name}_pivot_link" />
             </joint>
-            <actuator name="${name}_pivot_motor">
-                <hardwareInterface>hardware_interface/EffortJointInterface</hardwareInterface>
-                <mechanicalReduction>1</mechanicalReduction>
-            </actuator>
-        </transmission>
+            <transmission name="${name}_pivot_transmission">
+                <type>transmission_interface/SimpleTransmission</type>
+                <joint name="${name}_pivot_caster_joint">
+                    <hardwareInterface>hardware_interface/EffortJointInterface</hardwareInterface>
+                </joint>
+                <actuator name="${name}_pivot_motor">
+                    <hardwareInterface>hardware_interface/EffortJointInterface</hardwareInterface>
+                    <mechanicalReduction>1</mechanicalReduction>
+                </actuator>
+            </transmission>
+        </xacro:if>
+        <xacro:unless value="${movable_joints}">
+            <joint name="${name}_pivot_caster_joint" type="fixed">
+                <xacro:insert_block name="origin" />
+                <axis xyz="0 0 1"/>
+                <parent link="${parent}"/>
+                <child link="${name}_pivot_link" />
+            </joint>
+        </xacro:unless>
         <link name="${name}_pivot_link">
             <visual>
@@ -68,20 +78,30 @@
         </link>
         <!-- CASTER WHEEL -->
-        <joint name="${name}_wheel_joint" type="continuous">
-            <origin xyz="0 0 0" rpy="0 0 0"/>
-            <axis xyz="0 1 0"/>
-            <parent link="${name}_caster_offset_link"/>
-            <child link="${name}_wheel_link" />
-        </joint>
-        <transmission name="${name}_wheel_transmission">
-            <type>transmission_interface/SimpleTransmission</type>
-            <joint name="${name}_wheel_joint">
-                <hardwareInterface>hardware_interface/EffortJointInterface</hardwareInterface>
+        <xacro:if value="${movable_joints}">
+            <joint name="${name}_wheel_joint" type="continuous">
+                <origin xyz="0 0 0" rpy="0 0 0"/>
+                <axis xyz="0 1 0"/>
+                <parent link="${name}_caster_offset_link"/>
+                <child link="${name}_wheel_link" />
             </joint>
-            <actuator name="${name}_wheel_motor">
-                <hardwareInterface>hardware_interface/EffortJointInterface</hardwareInterface>
-                <mechanicalReduction>1</mechanicalReduction>
-            </actuator>
-        </transmission>
+            <transmission name="${name}_wheel_transmission">
+                <type>transmission_interface/SimpleTransmission</type>
+                <joint name="${name}_wheel_joint">
+                    <hardwareInterface>hardware_interface/EffortJointInterface</hardwareInterface>
+                </joint>
+                <actuator name="${name}_wheel_motor">
+                    <hardwareInterface>hardware_interface/EffortJointInterface</hardwareInterface>
+                    <mechanicalReduction>1</mechanicalReduction>
+                </actuator>
+            </transmission>
+        </xacro:if>
+        <xacro:unless value="${movable_joints}">
+            <joint name="${name}_wheel_joint" type="fixed">
+                <origin xyz="0 0 0" rpy="0 0 0"/>
+                <axis xyz="0 1 0"/>
+                <parent link="${name}_caster_offset_link"/>
+                <child link="${name}_wheel_link" />
+            </joint>
+        </xacro:unless>
         <link name="${name}_wheel_link">
             <visual>

File: urdf/robile_bricks/robile_active_wheel_brick.urdf.xacro (robot description, xacro)
@@ -30,5 +30,5 @@
 -->
 <robot xmlns:xacro="http://www.ros.org/wiki/xacro">
-    <xacro:macro name="robile_active_wheel_brick" params="name parent *origin">
+    <xacro:macro name="robile_active_wheel_brick" params="name parent *origin movable_joints:=true">
         <!-- Include xacro files-->
         <xacro:include filename="$(find robile_description)/urdf/base_macros/brick_housing.urdf.xacro" />
@@ -40,5 +40,5 @@
         </joint>
         <xacro:brick_housing name="${name}" with_wheel="true" color="red"/>
-        <xacro:kelo_drive name="${name}_drive" parent="${name}_link">
+        <xacro:kelo_drive name="${name}_drive" parent="${name}_link" movable_joints="${movable_joints}">
             <origin xyz="0 0 0" rpy="0 0 0.0"/>
         </xacro:kelo_drive>

File: urdf/robile_bricks/robile_passive_wheel_brick.urdf.xacro (robot description, xacro)
@@ -30,5 +30,5 @@
 -->
 <robot xmlns:xacro="http://www.ros.org/wiki/xacro">
-    <xacro:macro name="robile_passive_wheel_brick" params="name parent *origin">
+    <xacro:macro name="robile_passive_wheel_brick" params="name parent *origin movable_joints:=true">
         <!-- Include xacro files-->
         <xacro:include filename="$(find robile_description)/urdf/base_macros/brick_housing.urdf.xacro" />
@@ -40,5 +40,5 @@
         </joint>
         <xacro:brick_housing name="${name}" with_wheel="true" color="blue"/>
-        <xacro:passive_caster_wheel name="${name}_caster_wheel" parent="${name}_link">
+        <xacro:passive_caster_wheel name="${name}_caster_wheel" parent="${name}_link" movable_joints="${movable_joints}">
             <origin xyz="0 0 0" rpy="0 0 0.0"/>
         </xacro:passive_caster_wheel>
