Commit message: [4_wheel_lidar_config] Updates and fixes

File: robots/4_wheel_lidar_config.urdf.xacro (robot description, xacro)
@@ -1,5 +1,5 @@
 <?xml version='1.0'?>
 <!--
-Copyright (c) 2021
+Copyright (c) 2022
 KELO Robotics GmbH
 Author:
@@ -30,5 +30,6 @@
 License LGPL and BSD license along with this program.
 -->
-<robot xmlns:xacro="http://ros.org/wiki/xacro" name="4_wheel_config" >
+<robot xmlns:xacro="http://ros.org/wiki/xacro" name="4_wheel_lidar_config" >
+    <xacro:arg name="movable_joints" default="true"/>
     <!-- Include desired robile bricks -->
     <xacro:include filename="$(find robile_description)/urdf/robile_bricks/robile_active_wheel_brick.urdf.xacro" />
@@ -38,8 +39,8 @@
     <link name="base_link"/>
     <!-- Build platform using robile bricks -->
-    <xacro:robile_active_wheel_brick name="robile_1" parent="base_link">
+    <xacro:robile_active_wheel_brick name="robile_1" parent="base_link" movable_joints="$(arg movable_joints)">
         <origin xyz="0.233 0.1165 0.05" rpy="0.0 0.0 0.0"/>
     </xacro:robile_active_wheel_brick>
-    <xacro:robile_active_wheel_brick name="robile_2" parent="base_link">
+    <xacro:robile_active_wheel_brick name="robile_2" parent="base_link" movable_joints="$(arg movable_joints)">
         <origin xyz="0.233 -0.1165 0.05" rpy="0.0 0.0 0.0"/>
     </xacro:robile_active_wheel_brick>
@@ -50,13 +51,13 @@
         <origin xyz="0.0 -0.1165 0.05" rpy="0.0 0.0 0.0"/>
     </xacro:robile_master_battery_brick>
-    <xacro:robile_active_wheel_brick name="robile_5" parent="base_link">
+    <xacro:robile_active_wheel_brick name="robile_5" parent="base_link" movable_joints="$(arg movable_joints)">
         <origin xyz="-0.233 0.1165 0.05" rpy="0.0 0.0 0.0"/>
     </xacro:robile_active_wheel_brick>
-    <xacro:robile_active_wheel_brick name="robile_6" parent="base_link">
+    <xacro:robile_active_wheel_brick name="robile_6" parent="base_link" movable_joints="$(arg movable_joints)">
         <origin xyz="-0.233 -0.1165 0.05" rpy="0.0 0.0 0.0"/>
     </xacro:robile_active_wheel_brick>
-    <!-- SICK LASER -->
+    <!-- Datalogic LASER -->
     <xacro:datalogic name="base_laser_front" parent="base_link" topic="base_scan">
-        <origin xyz="0.42 0.0 0.35" rpy="0 0 0"/>
+        <origin xyz="0.43 0.0 0.32" rpy="0 0 0"/>
     </xacro:datalogic>
 </robot>

File: urdf/sensors/datalogic.urdf.xacro (robot description, xacro)
@@ -28,6 +28,11 @@
 <robot xmlns:xacro="http://www.ros.org/wiki/xacro">
     <xacro:include filename="$(find robile_description)/urdf/sensors/common.xacro" />
-    <xacro:macro name="datalogic" params="*origin name:=base_laser_front topic:=base_scan parent:=base_link sample_size:=540 update_rate:=10
-    min_angle:=-2.35619 max_angle:=2.35619 min_range:=0.1 max_range:=30.0 robot_namespace:=/ use_gpu:=true visualize:=false" >
+    <xacro:macro name="datalogic" params="*origin name:=base_laser_front
+                                          topic:=base_scan parent:=base_link
+                                          sample_size:=540 update_rate:=10
+                                          min_angle:=-2.35619 max_angle:=2.35619
+                                          min_range:=0.1 max_range:=30.0
+                                          robot_namespace:=/ use_gpu:=true
+                                          visualize:=false" >
         <joint name="${name}_joint" type="fixed">
             <axis xyz="0 1 0" />
@@ -39,5 +44,4 @@
             <inertial>
                 <mass value="1.1" />
-                <!-- <origin xyz="0 0 0" /> -->
                 <origin xyz="0 0 -0.05" rpy="0 0 0" />
                 <inertia ixx="${0.0833333 * 1.1 * (0.102*0.102 + 0.152*0.152)}" ixy="0.0" ixz="0.0"
@@ -46,5 +50,5 @@
             </inertial>
             <visual>
-                <origin xyz="-0.1 -0.08 0" rpy="0 0 3.14159" />
+                <origin xyz="-0.1 -0.08 -0.05" rpy="0 0 3.14159" />
                 <geometry>
                     <!-- Origin of this mesh is the focal point of the LIDAR. -->
@@ -53,7 +57,7 @@
             </visual>
             <collision>
-                <origin xyz="0 0 -0.05" rpy="0 0 0" />
+                <origin xyz="-0.025 0 -0.025" rpy="0 0 0" />
                 <geometry>
-                    <box size="0.105 0.1 0.1" />
+                    <box size="0.105 0.1 0.15" />
                 </geometry>
             </collision>
