Commit message: Rename caster_wheel -> passive_caster_wheel

File: urdf/base_macros/passive_caster_wheel.urdf.xacro (robot description, xacro)
@@ -30,5 +30,5 @@
 -->
 <robot xmlns:xacro="http://www.ros.org/wiki/xacro">
-    <xacro:macro name="caster_wheel" params="name parent *origin">
+    <xacro:macro name="passive_caster_wheel" params="name parent *origin">
         <xacro:include filename="$(find robile_description)/urdf/base_macros/common.xacro" />
         <!-- PIVOT -->
@@ -53,5 +53,5 @@
                 <origin xyz="0 0 0" rpy="0 0 0"/>
                 <geometry>
-                    <mesh filename="package://robile_description/meshes/caster_wheel/pivot.dae" scale="1 1 1"/>
+                    <mesh filename="package://robile_description/meshes/passive_caster_wheel/pivot.dae" scale="1 1 1"/>
                 </geometry>
             </visual>
@@ -88,5 +88,5 @@
                 <origin xyz="-0.031557 0.00007 0.0" rpy="0 0 0"/>
                 <geometry>
-                    <mesh filename="package://robile_description/meshes/caster_wheel/wheel.dae" scale="1 1 1"/>
+                    <mesh filename="package://robile_description/meshes/passive_caster_wheel/wheel.dae" scale="1 1 1"/>
                 </geometry>
             </visual>

File: urdf/robile_bricks/robile_passive_wheel_brick.urdf.xacro (robot description, xacro)
@@ -33,5 +33,5 @@
         <!-- Include xacro files-->
         <xacro:include filename="$(find robile_description)/urdf/base_macros/brick_housing.urdf.xacro" />
-        <xacro:include filename="$(find robile_description)/urdf/base_macros/caster_wheel.urdf.xacro" />
+        <xacro:include filename="$(find robile_description)/urdf/base_macros/passive_caster_wheel.urdf.xacro" />
         <joint name="${name}_joint" type="fixed">
             <xacro:insert_block name="origin" />
@@ -40,7 +40,7 @@
         </joint>
         <xacro:brick_housing name="${name}" with_wheel="true" color="blue"/>
-        <xacro:caster_wheel name="${name}_caster_wheel" parent="${name}_link">
+        <xacro:passive_caster_wheel name="${name}_caster_wheel" parent="${name}_link">
             <origin xyz="0 0 0" rpy="0 0 0.0"/>
-        </xacro:caster_wheel>
+        </xacro:passive_caster_wheel>
     </xacro:macro>
 </robot>
