Commit message: Rename robile_body -> brick_housing

File: urdf/base_macros/brick_housing.urdf.xacro (robot description, xacro)
@@ -30,5 +30,5 @@
 -->
 <robot xmlns:xacro="http://www.ros.org/wiki/xacro">
-    <xacro:macro name="robile_body" params="name color:=yellow with_wheel:=false">
+    <xacro:macro name="brick_housing" params="name color:=yellow with_wheel:=false">
         <!-- Include required xacro files -->
         <xacro:include filename="$(find robile_description)/urdf/base_macros/common.xacro" />
@@ -46,8 +46,8 @@
                 <geometry>
                     <xacro:if value="${with_wheel}">
-                        <mesh filename="package://robile_description/meshes/robile/wheeled_robile_body.dae" scale="1 1 1"/>
+                        <mesh filename="package://robile_description/meshes/robile_brick_housing/wheeled_brick_housing.dae" scale="1 1 1"/>
                     </xacro:if>
                     <xacro:unless value="${with_wheel}">
-                        <mesh filename="package://robile_description/meshes/robile/general_robile_body.dae" scale="1 1 1"/>
+                        <mesh filename="package://robile_description/meshes/robile_brick_housing/general_brick_housing.dae" scale="1 1 1"/>
                     </xacro:unless>
                 </geometry>
@@ -57,5 +57,5 @@
                 <origin xyz="0 0 0" rpy="0 0 0"/>
                 <geometry>
-                    <mesh filename="package://robile_description/meshes/robile/robile_lid.dae" scale="1 1 1"/>
+                    <mesh filename="package://robile_description/meshes/robile_brick_housing/lid.dae" scale="1 1 1"/>
                 </geometry>
             </visual>
@@ -64,8 +64,8 @@
                 <origin xyz="0 0 0" rpy="0 0 0"/>
                 <geometry>
-                    <mesh filename="package://robile_description/meshes/robile/robile_lid_cover_${color}.dae" scale="1 1 1"/>
+                    <mesh filename="package://robile_description/meshes/robile_brick_housing/lid_cover_${color}.dae" scale="1 1 1"/>
                 </geometry>
             </visual>
-            <!-- Collision box for robile body -->
+            <!-- Collision box for brick housing -->
             <collision>
                 <origin xyz="${center_of_mass_x} ${center_of_mass_y} ${center_of_mass_z}" rpy="0 0 0"/>
@@ -74,5 +74,5 @@
                 </geometry>
             </collision>
-            <!-- Inertia for robile body -->
+            <!-- Inertia for brick housing -->
             <xacro:cuboid_inertia mass="5.0"
                                 length="${robile_size_x}"

File: urdf/robile_bricks/robile_active_wheel_brick.urdf.xacro (robot description, xacro)
@@ -32,5 +32,5 @@
     <xacro:macro name="robile_active_wheel_brick" params="name parent *origin">
         <!-- Include xacro files-->
-        <xacro:include filename="$(find robile_description)/urdf/base_macros/robile_body.urdf.xacro" />
+        <xacro:include filename="$(find robile_description)/urdf/base_macros/brick_housing.urdf.xacro" />
         <xacro:include filename="$(find robile_description)/urdf/base_macros/kelo_drive.urdf.xacro" />
         <joint name="${name}_joint" type="fixed">
@@ -39,5 +39,5 @@
             <child link="${name}_link" />
         </joint>
-        <xacro:robile_body name="${name}" with_wheel="true" color="red"/>
+        <xacro:brick_housing name="${name}" with_wheel="true" color="red"/>
         <xacro:kelo_drive name="${name}_drive" parent="${name}_link">
             <origin xyz="0 0 0" rpy="0 0 0.0"/>

File: urdf/robile_bricks/robile_cpu_brick.urdf.xacro (robot description, xacro)
@@ -31,5 +31,5 @@
 <robot xmlns:xacro="http://www.ros.org/wiki/xacro">
     <xacro:macro name="robile_cpu_brick" params="name parent *origin">
-        <xacro:include filename="$(find robile_description)/urdf/base_macros/robile_body.urdf.xacro" />
+        <xacro:include filename="$(find robile_description)/urdf/base_macros/brick_housing.urdf.xacro" />
         <joint name="${name}_joint" type="fixed">
             <xacro:insert_block name="origin" />
@@ -37,5 +37,5 @@
             <child link="${name}_link" />
         </joint>
-        <xacro:robile_body name="${name}"/>
+        <xacro:brick_housing name="${name}"/>
     </xacro:macro>
 </robot>

File: urdf/robile_bricks/robile_empty_brick.urdf.xacro (robot description, xacro)
@@ -31,5 +31,5 @@
 <robot xmlns:xacro="http://www.ros.org/wiki/xacro">
     <xacro:macro name="robile_empty_brick" params="name parent *origin">
-        <xacro:include filename="$(find robile_description)/urdf/base_macros/robile_body.urdf.xacro" />
+        <xacro:include filename="$(find robile_description)/urdf/base_macros/brick_housing.urdf.xacro" />
         <joint name="${name}_joint" type="fixed">
             <xacro:insert_block name="origin" />
@@ -37,5 +37,5 @@
             <child link="${name}_link" />
         </joint>
-        <xacro:robile_body name="${name}" color="blue"/>
+        <xacro:brick_housing name="${name}" color="blue"/>
     </xacro:macro>
 </robot>

File: urdf/robile_bricks/robile_master_battery_brick.urdf.xacro (robot description, xacro)
@@ -31,5 +31,5 @@
 <robot xmlns:xacro="http://www.ros.org/wiki/xacro">
     <xacro:macro name="robile_master_battery_brick" params="name parent *origin">
-        <xacro:include filename="$(find robile_description)/urdf/base_macros/robile_body.urdf.xacro" />
+        <xacro:include filename="$(find robile_description)/urdf/base_macros/brick_housing.urdf.xacro" />
         <joint name="${name}_joint" type="fixed">
             <xacro:insert_block name="origin" />
@@ -37,5 +37,5 @@
             <child link="${name}_link" />
         </joint>
-        <xacro:robile_body name="${name}" color="green"/>
+        <xacro:brick_housing name="${name}" color="green"/>
     </xacro:macro>
 </robot>

File: urdf/robile_bricks/robile_passive_wheel_brick.urdf.xacro (robot description, xacro)
@@ -32,5 +32,5 @@
     <xacro:macro name="robile_passive_wheel_brick" params="name parent *origin">
         <!-- Include xacro files-->
-        <xacro:include filename="$(find robile_description)/urdf/base_macros/robile_body.urdf.xacro" />
+        <xacro:include filename="$(find robile_description)/urdf/base_macros/brick_housing.urdf.xacro" />
         <xacro:include filename="$(find robile_description)/urdf/base_macros/caster_wheel.urdf.xacro" />
         <joint name="${name}_joint" type="fixed">
@@ -39,5 +39,5 @@
             <child link="${name}_link" />
         </joint>
-        <xacro:robile_body name="${name}" with_wheel="true" color="blue"/>
+        <xacro:brick_housing name="${name}" with_wheel="true" color="blue"/>
         <xacro:caster_wheel name="${name}_caster_wheel" parent="${name}_link">
             <origin xyz="0 0 0" rpy="0 0 0.0"/>

File: urdf/robile_bricks/robile_slave_battery_brick.urdf.xacro (robot description, xacro)
@@ -31,5 +31,5 @@
 <robot xmlns:xacro="http://www.ros.org/wiki/xacro">
     <xacro:macro name="robile_slave_battery_brick" params="name parent *origin">
-        <xacro:include filename="$(find robile_description)/urdf/base_macros/robile_body.urdf.xacro" />
+        <xacro:include filename="$(find robile_description)/urdf/base_macros/brick_housing.urdf.xacro" />
         <joint name="${name}_joint" type="fixed">
             <xacro:insert_block name="origin" />
@@ -37,5 +37,5 @@
             <child link="${name}_link" />
         </joint>
-        <xacro:robile_body name="${name}" color="green"/>
+        <xacro:brick_housing name="${name}" color="green"/>
     </xacro:macro>
 </robot>

Commit message: update bricks to use more accurate inertia and collision block

File: urdf/base_macros/brick_housing.urdf.xacro (robot description, xacro)
@@ -37,7 +37,4 @@
         <xacro:property name="robile_size_y" value="0.233"/>
         <xacro:property name="robile_size_z" value="0.239"/>
-        <xacro:property name="center_of_mass_x" value="0.0005"/>
-        <xacro:property name="center_of_mass_y" value="0.0001"/>
-        <xacro:property name="center_of_mass_z" value="0.119"/>
         <link name="${name}_link">
             <!-- Aluminium casing of the robile -->
@@ -69,5 +66,5 @@
             <!-- Collision box for brick housing -->
             <collision>
-                <origin xyz="${center_of_mass_x} ${center_of_mass_y} ${center_of_mass_z}" rpy="0 0 0"/>
+                <origin xyz="0 0 ${robile_size_z/2}" rpy="0 0 0"/>
                 <geometry>
                     <box size="${robile_size_x} ${robile_size_y} ${robile_size_z}" />
@@ -75,11 +72,18 @@
             </collision>
             <!-- Inertia for brick housing -->
-            <xacro:cuboid_inertia mass="5.0"
-                                length="${robile_size_x}"
-                                breadth="${robile_size_y}"
-                                height="${robile_size_z}"
-                                center_of_mass_x="${center_of_mass_x}"
-                                center_of_mass_y="${center_of_mass_y}"
-                                center_of_mass_z="${center_of_mass_z}"/>
+            <xacro:if value="${with_wheel}">
+                <inertial>
+                    <mass value="4.554" />
+                    <origin xyz="0.00005 0.00009 0.12048" />
+                    <inertia  ixx="0.0512" ixy="0.0000062" ixz="0.0000224" iyy="0.051012" iyz="0.000027" izz="0.062741" />
+                </inertial>
+            </xacro:if>
+            <xacro:unless value="${with_wheel}">
+                <inertial>
+                    <mass value="4.554" />
+                    <origin xyz="0.00005 0.00009 0.12048" />
+                    <inertia  ixx="0.0512" ixy="0.0000062" ixz="0.0000224" iyy="0.051012" iyz="0.000027" izz="0.062741" />
+                </inertial>
+		    </xacro:unless>
         </link>
     </xacro:macro>

File: urdf/base_macros/kelo_drive_wheel.urdf.xacro (robot description, xacro)
@@ -71,5 +71,12 @@
                 </geometry>
             </collision>
-            <!-- <xacro:cylinder_inertia mass="0.5" radius="0.0515" length="0.035" center_of_mass_roll="1.570796327"/> -->
+            <!-- xacro:cylinder_inertia mass="0.5" radius="0.0515" length="0.035" center_of_mass_roll="1.570796327"/ -->
+<!--
+            <inertial>
+                <mass value="2.0829" />
+                <origin xyz="0 0.00038 -0.00002" />
+                <inertia  ixx="0.001385" ixy="0" ixz="0" iyy="0.001998" iyz="-0.0000005" izz="0.0013857" />
+            </inertial>
+-->
             <!--HACK: Use large cuboid inertias to fix the issue that the model breaks when JointVelocity controller is activated -->
             <xacro:cuboid_inertia mass="10.0" length="0.233" breadth="0.233" height="0.233"/>

File: urdf/robile_bricks/robile_cpu_brick.urdf.xacro (robot description, xacro)
@@ -31,5 +31,9 @@
 <robot xmlns:xacro="http://www.ros.org/wiki/xacro">
     <xacro:macro name="robile_cpu_brick" params="name parent *origin">
-        <xacro:include filename="$(find robile_description)/urdf/base_macros/brick_housing.urdf.xacro" />
+        <!-- Properties for cpu brick -->
+        <xacro:property name="color" value="yellow"/>
+        <xacro:property name="robile_size_x" value="0.233"/>
+        <xacro:property name="robile_size_y" value="0.233"/>
+        <xacro:property name="robile_size_z" value="0.239"/>
         <joint name="${name}_joint" type="fixed">
             <xacro:insert_block name="origin" />
@@ -37,5 +41,40 @@
             <child link="${name}_link" />
         </joint>
-        <xacro:brick_housing name="${name}"/>
+        <link name="${name}_link">
+            <!-- Aluminium casing -->
+            <visual>
+                <origin xyz="0 0 0" rpy="0 0 0"/>
+                <geometry>
+                    <mesh filename="package://robile_description/meshes/robile_brick_housing/general_brick_housing.dae" scale="1 1 1"/>
+                </geometry>
+            </visual>
+            <!-- robile lid -->
+            <visual>
+                <origin xyz="0 0 0" rpy="0 0 0"/>
+                <geometry>
+                    <mesh filename="package://robile_description/meshes/robile_brick_housing/lid.dae" scale="1 1 1"/>
+                </geometry>
+            </visual>
+            <!-- robile lid cover (color passed as a parameter) -->
+            <visual>
+                <origin xyz="0 0 0" rpy="0 0 0"/>
+                <geometry>
+                    <mesh filename="package://robile_description/meshes/robile_brick_housing/lid_cover_${color}.dae" scale="1 1 1"/>
+                </geometry>
+            </visual>
+            <!-- Collision box for brick housing -->
+            <collision>
+                <origin xyz="0 0 ${robile_size_z/2}" rpy="0 0 0"/>
+                <geometry>
+                    <box size="${robile_size_x} ${robile_size_y} ${robile_size_z}" />
+                </geometry>
+            </collision>
+            <!-- Inertia for cpu brick -->
+            <inertial>
+                <mass value="6.44075" />
+                <origin xyz="0.00413 0.0053 0.10792" />
+                <inertia  ixx="0.059819" ixy="0.000584" ixz="-0.000138" iyy="0.059845" iyz="-0.000069" izz="0.06767" />
+            </inertial>
+        </link>
     </xacro:macro>
 </robot>

File: urdf/robile_bricks/robile_master_battery_brick.urdf.xacro (robot description, xacro)
@@ -31,5 +31,9 @@
 <robot xmlns:xacro="http://www.ros.org/wiki/xacro">
     <xacro:macro name="robile_master_battery_brick" params="name parent *origin">
-        <xacro:include filename="$(find robile_description)/urdf/base_macros/brick_housing.urdf.xacro" />
+        <!-- Properties for master battery brick -->
+        <xacro:property name="color" value="green"/>
+        <xacro:property name="robile_size_x" value="0.233"/>
+        <xacro:property name="robile_size_y" value="0.233"/>
+        <xacro:property name="robile_size_z" value="0.239"/>
         <joint name="${name}_joint" type="fixed">
             <xacro:insert_block name="origin" />
@@ -37,5 +41,40 @@
             <child link="${name}_link" />
         </joint>
-        <xacro:brick_housing name="${name}" color="green"/>
+        <link name="${name}_link">
+            <!-- Aluminium casing -->
+            <visual>
+                <origin xyz="0 0 0" rpy="0 0 0"/>
+                <geometry>
+                    <mesh filename="package://robile_description/meshes/robile_brick_housing/general_brick_housing.dae" scale="1 1 1"/>
+                </geometry>
+            </visual>
+            <!-- robile lid -->
+            <visual>
+                <origin xyz="0 0 0" rpy="0 0 0"/>
+                <geometry>
+                    <mesh filename="package://robile_description/meshes/robile_brick_housing/lid.dae" scale="1 1 1"/>
+                </geometry>
+            </visual>
+            <!-- robile lid cover (color passed as a parameter) -->
+            <visual>
+                <origin xyz="0 0 0" rpy="0 0 0"/>
+                <geometry>
+                    <mesh filename="package://robile_description/meshes/robile_brick_housing/lid_cover_${color}.dae" scale="1 1 1"/>
+                </geometry>
+            </visual>
+            <!-- Collision box for brick housing -->
+            <collision>
+                <origin xyz="0 0 ${robile_size_z/2}" rpy="0 0 0"/>
+                <geometry>
+                    <box size="${robile_size_x} ${robile_size_y} ${robile_size_z}" />
+                </geometry>
+            </collision>
+            <!-- Inertia for master battery brick -->
+            <inertial>
+                <mass value="11.649" />
+                <origin xyz="0 -0.00012 0.09665" />
+                <inertia  ixx="0.090592" ixy="-0.0000008" ixz="0.000011" iyy="0.097288" iyz="0.000217" izz="0.101994" />
+            </inertial>
+        </link>
     </xacro:macro>
 </robot>

File: urdf/robile_bricks/robile_slave_battery_brick.urdf.xacro (robot description, xacro)
@@ -31,5 +31,9 @@
 <robot xmlns:xacro="http://www.ros.org/wiki/xacro">
     <xacro:macro name="robile_slave_battery_brick" params="name parent *origin">
-        <xacro:include filename="$(find robile_description)/urdf/base_macros/brick_housing.urdf.xacro" />
+        <!-- Properties for slave battery brick -->
+        <xacro:property name="color" value="green"/>
+        <xacro:property name="robile_size_x" value="0.233"/>
+        <xacro:property name="robile_size_y" value="0.233"/>
+        <xacro:property name="robile_size_z" value="0.239"/>
         <joint name="${name}_joint" type="fixed">
             <xacro:insert_block name="origin" />
@@ -37,5 +41,40 @@
             <child link="${name}_link" />
         </joint>
-        <xacro:brick_housing name="${name}" color="green"/>
+        <link name="${name}_link">
+            <!-- Aluminium casing -->
+            <visual>
+                <origin xyz="0 0 0" rpy="0 0 0"/>
+                <geometry>
+                    <mesh filename="package://robile_description/meshes/robile_brick_housing/general_brick_housing.dae" scale="1 1 1"/>
+                </geometry>
+            </visual>
+            <!-- robile lid -->
+            <visual>
+                <origin xyz="0 0 0" rpy="0 0 0"/>
+                <geometry>
+                    <mesh filename="package://robile_description/meshes/robile_brick_housing/lid.dae" scale="1 1 1"/>
+                </geometry>
+            </visual>
+            <!-- robile lid cover (color passed as a parameter) -->
+            <visual>
+                <origin xyz="0 0 0" rpy="0 0 0"/>
+                <geometry>
+                    <mesh filename="package://robile_description/meshes/robile_brick_housing/lid_cover_${color}.dae" scale="1 1 1"/>
+                </geometry>
+            </visual>
+            <!-- Collision box for brick housing -->
+            <collision>
+                <origin xyz="0 0 ${robile_size_z/2}" rpy="0 0 0"/>
+                <geometry>
+                    <box size="${robile_size_x} ${robile_size_y} ${robile_size_z}" />
+                </geometry>
+            </collision>
+            <!-- Inertia for slave battery brick -->
+            <inertial>
+                <mass value="11.649" />
+                <origin xyz="0 -0.00012 0.09665" />
+                <inertia  ixx="0.090592" ixy="-0.0000008" ixz="0.000011" iyy="0.097288" iyz="0.000217" izz="0.101994" />
+            </inertial>
+        </link>
     </xacro:macro>
 </robot>
