Commit message: Rename kelo_hub_wheel -> kelo_drive_wheel

File: urdf/base_macros/kelo_drive.urdf.xacro (robot description, xacro)
@@ -32,5 +32,5 @@
     <xacro:macro name="kelo_drive" params="name parent *origin">
         <xacro:include filename="$(find robile_description)/urdf/base_macros/common.xacro" />
-        <xacro:include filename="$(find robile_description)/urdf/base_macros/kelo_hub_wheel.urdf.xacro" />
+        <xacro:include filename="$(find robile_description)/urdf/base_macros/kelo_drive_wheel.urdf.xacro" />
         <!-- PIVOT -->
         <joint name="${name}_pivot_joint" type="continuous">
@@ -68,11 +68,11 @@
         </link>
         <!-- LEFT HUB WHEEL -->
-        <xacro:kelo_hub_wheel name="${name}_left_hub_wheel" parent="${name}_pivot_link">
+        <xacro:kelo_drive_wheel name="${name}_left_hub_wheel" parent="${name}_pivot_link">
             <origin xyz="0 0.039326 0.001514" rpy="0 0 0.0"/>
-        </xacro:kelo_hub_wheel>
+        </xacro:kelo_drive_wheel>
         <!-- RIGHT HUB WHEEL -->
-        <xacro:kelo_hub_wheel name="${name}_right_hub_wheel" parent="${name}_pivot_link">
+        <xacro:kelo_drive_wheel name="${name}_right_hub_wheel" parent="${name}_pivot_link">
             <origin xyz="0 -0.039326 0.001514" rpy="0 0 0.0"/>
-        </xacro:kelo_hub_wheel>
+        </xacro:kelo_drive_wheel>
     </xacro:macro>
 </robot>

File: urdf/base_macros/kelo_drive_wheel.urdf.xacro (robot description, xacro)
@@ -30,5 +30,5 @@
 -->
 <robot xmlns:xacro="http://www.ros.org/wiki/xacro">
-    <xacro:macro name="kelo_hub_wheel" params="name parent *origin">
+    <xacro:macro name="kelo_drive_wheel" params="name parent *origin">
         <xacro:include filename="$(find robile_description)/urdf/base_macros/common.xacro" />
         <joint name="${name}_joint" type="continuous">
@@ -52,5 +52,5 @@
                 <origin xyz="0 0 0" rpy="0 0 0"/>
                 <geometry>
-                    <mesh filename="package://robile_description/meshes/kelo_drive/kelo_drive_hub_wheel.dae" scale="1 1 1"/>
+                    <mesh filename="package://robile_description/meshes/kelo_drive/kelo_drive_wheel.dae" scale="1 1 1"/>
                 </geometry>
             </visual>

Commit message: Add caster_offset for Kelo Drive

File: urdf/base_macros/kelo_drive.urdf.xacro (robot description, xacro)
@@ -69,9 +69,9 @@
         <!-- LEFT HUB WHEEL -->
         <xacro:kelo_drive_wheel name="${name}_left_hub_wheel" parent="${name}_pivot_link">
-            <origin xyz="0 0.039326 0.001514" rpy="0 0 0.0"/>
+            <origin xyz="-0.01 0.039326 0.001514" rpy="0 0 0.0"/>
         </xacro:kelo_drive_wheel>
         <!-- RIGHT HUB WHEEL -->
         <xacro:kelo_drive_wheel name="${name}_right_hub_wheel" parent="${name}_pivot_link">
-            <origin xyz="0 -0.039326 0.001514" rpy="0 0 0.0"/>
+            <origin xyz="-0.01 -0.039326 0.001514" rpy="0 0 0.0"/>
         </xacro:kelo_drive_wheel>
     </xacro:macro>

Commit message: update kelo drive inertia

File: urdf/base_macros/kelo_drive.urdf.xacro (robot description, xacro)
@@ -74,6 +74,9 @@
                 </geometry>
             </collision>
-            <!--TODO: Set the correct inertia-->
-            <xacro:cuboid_inertia mass="10.0" length="0.233" breadth="0.233" height="0.233"/>
+            <inertial>
+                <mass value="1.0006" />
+                <origin xyz="0.00034 -0.00046 0.0504" />
+                <inertia  ixx="0.0023" ixy="0.000008" ixz="0.000011" iyy="0.00249" iyz="-0.000014" izz="0.00288" />
+            </inertial>
         </link>
         <!-- LEFT HUB WHEEL -->

File: urdf/base_macros/kelo_drive_wheel.urdf.xacro (robot description, xacro)
@@ -71,5 +71,4 @@
                 </geometry>
             </collision>
-            <!-- xacro:cylinder_inertia mass="0.5" radius="0.0515" length="0.035" center_of_mass_roll="1.570796327"/ -->
 <!--
             <inertial>

Commit message: Revert "update kelo drive inertia"
This reverts commit 83e4a8700de01bef520c410c6a3643be0e4f867b.

File: urdf/base_macros/kelo_drive.urdf.xacro (robot description, xacro)
@@ -74,9 +74,6 @@
                 </geometry>
             </collision>
-            <inertial>
-                <mass value="1.0006" />
-                <origin xyz="0.00034 -0.00046 0.0504" />
-                <inertia  ixx="0.0023" ixy="0.000008" ixz="0.000011" iyy="0.00249" iyz="-0.000014" izz="0.00288" />
-            </inertial>
+            <!--TODO: Set the correct inertia-->
+            <xacro:cuboid_inertia mass="10.0" length="0.233" breadth="0.233" height="0.233"/>
         </link>
         <!-- LEFT HUB WHEEL -->

File: urdf/base_macros/kelo_drive_wheel.urdf.xacro (robot description, xacro)
@@ -71,4 +71,5 @@
                 </geometry>
             </collision>
+            <!-- xacro:cylinder_inertia mass="0.5" radius="0.0515" length="0.035" center_of_mass_roll="1.570796327"/ -->
 <!--
             <inertial>
