Commit message: add models

File: urdf/sensors/hokuyo_ust_10lx.urdf.xacro (robot description, xacro)
@@ -16,6 +16,6 @@
       <visual>
         <origin xyz="0 0 0" rpy="1.57 0 1.57" />
-      <geometry>
-        <mesh filename="package://robile_description/meshes/sensors/UST-10LX.dae" scale="1 1 1" />
+        <geometry>
+          <mesh filename="package://robile_description/meshes/sensors/UST-10LX.dae" scale="1 1 1" />
         </geometry>
       </visual>
